Commit message: fix(curt_mini_description): use package URIs for RViz meshes

File: curt_mini_description/models/curt_mini/robot.urdf.xacro (robot description, xacro)
@@ -25,5 +25,5 @@
       <origin xyz="0 0 0" rpy="0 0 0" />
       <geometry>
-        <mesh filename="file://$(arg path)/models/curt_mini/meshes/base_link.STL" />
+        <mesh filename="package://curt_mini_description/models/curt_mini/meshes/base_link.STL" />
       </geometry>
       <material name="">
@@ -34,5 +34,5 @@
       <origin xyz="0 0 0" rpy="0 0 0" />
       <geometry>
-        <mesh filename="file://$(arg path)/models/curt_mini/meshes/base_link.STL" />
+        <mesh filename="package://curt_mini_description/models/curt_mini/meshes/base_link.STL" />
       </geometry>
     </collision>
@@ -52,5 +52,5 @@
       <origin xyz="0 0 0" rpy="0 0 0" />
       <geometry>
-        <mesh filename="file://$(arg path)/models/curt_mini/meshes/wheel4_link.STL" />
+        <mesh filename="package://curt_mini_description/models/curt_mini/meshes/wheel4_link.STL" />
       </geometry>
       <material name="">
@@ -83,5 +83,5 @@
       <origin xyz="0 0 0" rpy="0 0 0" />
       <geometry>
-        <mesh filename="file://$(arg path)/models/curt_mini/meshes/wheel1_link.STL" />
+        <mesh filename="package://curt_mini_description/models/curt_mini/meshes/wheel1_link.STL" />
       </geometry>
       <material name="">
@@ -114,5 +114,5 @@
       <origin xyz="0 0 0" rpy="0 0 0" />
       <geometry>
-        <mesh filename="file://$(arg path)/models/curt_mini/meshes/wheel3_link.STL" />
+        <mesh filename="package://curt_mini_description/models/curt_mini/meshes/wheel3_link.STL" />
       </geometry>
       <material name="">
@@ -145,5 +145,5 @@
       <origin xyz="0 0 0" rpy="0 0 0" />
       <geometry>
-        <mesh filename="file://$(arg path)/models/curt_mini/meshes/wheel2_link.STL" />
+        <mesh filename="package://curt_mini_description/models/curt_mini/meshes/wheel2_link.STL" />
       </geometry>
       <material name="">
